File: master/PCB/LED Glasses Arm Board/LED Left Glasses Arm (mcu)/LED Left Glasses Arm (mcu).kicad_pcb (KiCad board)
At the start: 2 copper layers, 131.2 x 17.5 mm, 13 parts, among them J101 Front Connector, J102 SWD, SW101 Push Button, U101 MIC5504-3.3YM5, U102 STM32G071KBU6

Commit message: various changes made to mcu pcb
Parts:
- moved C105 4.87 mm to (133.5, 92.1), turned to 90 degrees
- moved SW101 4.41 mm to (137.7, 92.1), turned to 270 degrees
- moved C103 2.23 mm to (117.1, 91.7)
- moved C102 1.40 mm to (102.5, 92.2), turned to 90 degrees
- moved C101 1.00 mm to (96.1, 92.2), turned to 270 degrees
- moved U102 0.73 mm to (121.9, 91.7)
- moved R101 0.34 mm to (128.3, 92.0)
- turned C104 to 270 degrees
- turned MK101 to 0 degrees
- turned U101 to 90 degrees
Connections:
- U102 pad 31: Net-(U102-Pad31) -> /LED_DATA
- U102 pad 9: /LED_DATA -> Net-(U102-Pad9)
Routing:
- net GND: track 50.4 -> 8.33 mm, vias 5 -> 17
- net /NRST: track 34.9 -> 46.4 mm
- net +3V3: track 51.4 -> 58.4 mm, vias 0 -> 2
- net /MIC_MISO: track 14.0 -> 18.0 mm, vias 2 -> 0
- net /LED_DATA: track 36.0 -> 40.0 mm
- net /MIC_CLK: track 17.5 -> 13.7 mm
- net /SWCLK: track 26.7 -> 23.9 mm
- net /SWDIO: track 23.6 -> 24.6 mm
- net Net-(C101-Pad2): track 12.1 -> 11.3 mm
- added copper zone on F.Cu, net GND
Other:
- net class Default: via_dia 0.8 -> 0.7; via_drill 0.4 -> 0.5

Commit message: finished off the mcu arm pcb
Parts:
- added C106: 100n, 25V, Capacitor_SMD:C_0805_2012Metric_Pad1.15x1.40mm_HandSolder, F.Cu at (111.0, 92.0)
- added SW102: Push Button, Button_Switch_SMD:SW_SPST_CK_KXT3, F.Cu at (107.0, 92.0)
- moved C104 8.97 mm to (116.0, 92.0)
- moved R101 8.70 mm to (137.0, 92.0)
- moved MK101 8.62 mm to (119.5, 92.0)
- moved C105 8.50 mm to (142.0, 92.0)
- moved SW101 8.30 mm to (146.0, 92.0)
- moved U102 8.14 mm to (130.0, 92.0)
- moved C103 7.41 mm to (124.5, 92.0)
- moved J102 7.24 mm to (151.2, 91.0)
- moved J101 2.40 mm to (86.8, 93.6)
- moved D101 1.38 mm to (92.0, 93.0)
- moved C101 0.62 mm to (95.5, 92.0)
- moved U101 0.35 mm to (99.0, 92.0)
- moved C102 0.20 mm to (102.5, 92.0)
Routing:
- net Net-(C106-Pad1): track 0.00 -> 22.2 mm, vias 0 -> 4
- net +3V3: track 58.4 -> 71.4 mm
- net /LED_DATA: track 40.0 -> 47.0 mm
- net /NRST: track 46.4 -> 42.1 mm
- net /SWCLK: track 23.9 -> 27.1 mm
- net Net-(D101-Pad2): track 7.44 -> 4.78 mm
- net GND: track 8.33 -> 5.83 mm
- net /SWDIO: track 24.6 -> 26.1 mm
- net Net-(C101-Pad2): track 11.3 -> 10.4 mm
- net /MIC_MISO: track 18.0 -> 18.7 mm, vias 0 -> 2
- net /MIC_CLK: track 13.7 -> 13.8 mm, vias 2 -> 0
Other:
- net class Default: clearance 0.2 -> 0.15; trace_width 0.25 -> 0.15; via_dia 0.7 -> 0.45; via_drill 0.5 -> 0.3
- rule trace_clearance: 0.2 -> 0.15
- rule trace_min: 0.2 -> 0.15
- rule via_min_size: 0.4 -> 0.45
- board text added: "+"
- board text added: "-"
- board text added: "By Lamal and Dardy ©2020"
- board text added: "DATA"
- board text added: "NRST"
- board text added: "SWDIO"
